File: Silent Alarm Clock/V1/SilentAlarmClockPCB_V1/SilentAlarmClockPCB_V1.kicad_sch (KiCad schematic)
At the start: 28 parts, among them J1 USB_C_Receptacle_USB2.0_16P, J2 Barrel_Jack, J3 B2B-PH-K-S, SW1 BOOT, SW2 RESET, U2 ESP32-S3-MINI-1-N8, U3 BQ24040DSQR, U4 TLV75801PDRV, U5 ESD7104MUTAG

Commit message: fixed push button switch footprints
Parts:
- removed SW1: BOOT, Button_Switch_SMD:SW_SPST_PTS810, symbol Switch:SW_MEC_5E
- removed SW2: RESET, Button_Switch_SMD:SW_SPST_PTS810, symbol Switch:SW_MEC_5E
- added SW3: RESET, Button_Switch_SMD:SW_SPST_PTS810, symbol Switch:SW_Push
- added SW4: BOOT, Button_Switch_SMD:SW_SPST_PTS810, symbol Switch:SW_Push
Connections:
- net GND: now also SW3.1, SW4.1
- net at C9.1, R1.2, U2.45 (EN): now also SW3.2
- net at C10.1, U2.4 (IO0): now also SW4.2

Commit message: Finished V1 board
Parts:
- removed U5: ESD7104MUTAG, ESD7104MUTAG:IC_ESD7104MUTAG, symbol ESD7104MUTAG:ESD7104MUTAG
- added U1: ESD7104MUTAG, UDFN10_ONS, symbol ESD7104MUTAG:ESD7104MUTAG
Connections:
- net 3V3: now also C7.1, C8.1, R1.1, U2.3 (3V3)
- net 5VIN: now also U1.4 (I/O), U1.7 (NC)
- net GND: now also U1.3 (GND), U1.8 (GND)
- net USB_N: now also U1.2 (I/O), U1.9 (NC)
- net USB_P: now also U1.1 (I/O), U1.10 (NC)
