File: Silent Alarm Clock/V3/SilentAlarmClockPCB_V3/SilentAlarmClockPCB_V1.kicad_sch (KiCad schematic)
At the start: 46 parts, among them J1 USB_C_Receptacle_USB2.0_16P, J2 B2B-PH-K-S, J3 Conn_01x08_Socket, SW1 SW_SPDT, SW2 RotaryEncoder_Switch, SW3 RESET, SW4 BOOT, U1 BQ24075TRGTR, U2 ESP32-S3-MINI-1-N8, U3 TPS63001, U4 ESD7104MUTAG, U5 BQ27441DRZT-G1A

Commit message: Created V3 PCB step model
Parts:
- added H1, H2, H3, H4, H5, H6, H7, H8: MountingHole, symbol Mechanical:MountingHole
Other:
- note added: "Mounting Holes"
