File: Silent Alarm Clock/V3/SilentAlarmClockPCB_V3/SilentAlarmClockPCB_V1.kicad_pcb (KiCad board)
At the start: 4 copper layers, 92.5 x 70.4 mm, 46 parts, among them J1 USB_C_Receptacle_USB2.0_16P, J2 B2B-PH-K-S, J3 Conn_01x08_Socket, SW1 SW_SPDT, SW2 RotaryEncoder_Switch, U1 BQ24075TRGTR, U2 ESP32-S3-MINI-1-N8, U3 TPS63001, U4 ESD7104MUTAG, U5 BQ27441DRZT-G1A

Commit message: Created V3 PCB step model
Parts:
- added H2: MountingHole, MountingHole:MountingHole_4.3mm_M4, F.Cu at (186.5, 91.0)
- added H3: MountingHole, MountingHole:MountingHole_4.3mm_M4, F.Cu at (186.5, 128.0)
- added H4: MountingHole, MountingHole:MountingHole_4.3mm_M4, F.Cu at (139.0, 128.0)
- added H5: MountingHole, MountingHole:MountingHole_2.7mm_M2.5, F.Cu at (204.0, 120.0)
- added H6: MountingHole, MountingHole:MountingHole_2.7mm_M2.5, F.Cu at (204.0, 87.0)
- added H7: MountingHole, MountingHole:MountingHole_2.7mm_M2.5, F.Cu at (119.5, 87.0)
- added H8: MountingHole, MountingHole:MountingHole_2.7mm_M2.5, F.Cu at (119.5, 120.0)
- moved R2 9.34 mm to (128.2, 125.5)
- moved R3 9.34 mm to (128.2, 124.0)
- renumbered RESET to SW3, BOOT to SW4
Connections:
- U4 pad 7: V_USB -> unconnected-(U4-NC-Pad7)
- U5 pad 3: (no net) -> GND
- U5 pad V: GND -> (no net)
Routing:
- net CC2: track 11.9 -> 15.8 mm
- net CS: track 32.4 -> 36.2 mm
- net D-: track 57.3 -> 60.6 mm
- net GND: track 97.0 -> 94.3 mm
- net D+: track 58.7 -> 61.2 mm

Commit message: V3 PCB and Case Finished
Parts:
- removed H7, H8: MountingHole, MountingHole:MountingHole_2.7mm_M2.5
- added H1: MountingHole, MountingHole:MountingHole_4.3mm_M4, F.Cu at (150.5, 129.0)
- C6, C8, C9: value 1uF -> 10uF
- C7: value 1uF -> 0.1uF
- H3, H4: footprint MountingHole:MountingHole_4.3mm_M4 -> MountingHole:MountingHole_2.7mm_M2.5
- J2: moved to B.Cu
- R16: value 10k -> 100
- R7: value 440 -> 1.1k
- moved H6 84.5 mm to (119.5, 87.0)
- moved H4 76.9 mm to (204.0, 87.0)
- moved J3 68.3 mm to (180.0, 130.0), turned to 0 degrees
- moved H3 67.5 mm to (119.5, 120.0)
- moved H2 40.7 mm to (172.0, 129.0)
- turned J2 to -90 degrees
Connections:
- U1 pad V: (no net) -> GND
- U4 pad 7: unconnected-(U4-NC-Pad7) -> V_USB
- U5 pad V: (no net) -> GND
Routing:
- net CS: track 36.2 -> 94.5 mm, vias 0 -> 2
- net 3V3: track 39.9 -> 95.0 mm, vias 13 -> 15
- net DIN: track 25.5 -> 80.0 mm, vias 0 -> 2
- net CLK: track 26.8 -> 79.2 mm, vias 0 -> 2
- net D/C: track 31.1 -> 82.0 mm, vias 0 -> 2
- net RST: track 33.5 -> 82.7 mm, vias 0 -> 2
- net BUSY: track 35.8 -> 83.8 mm, vias 0 -> 2
- net OUT: track 14.5 -> 33.0 mm
- net BATTERY_IN: track 63.8 -> 71.7 mm
- net GND: track 94.3 -> 88.3 mm
