File: Silent Alarm Clock/V3/SilentAlarmClockPCB_V3/_restore_backup_2026-08-10T11-58-46-238/SilentAlarmClockPCB_V1.kicad_sch (KiCad schematic)
At the start: 52 parts, among them J1 USB_C_Receptacle_USB2.0_16P, J2 B2B-PH-K-S, J3 Conn_01x08_Socket, SW1 SW_SPDT, SW2 RotaryEncoder_Switch, SW3 RESET, SW4 BOOT, U1 BQ24075TRGTR, U2 ESP32-S3-MINI-1-N8, U3 TPS63001, U4 ESD7104MUTAG, U5 BQ27441DRZT-G1A

Commit message: V3 PCB and Case Finished
Parts:
- added H7, H8: MountingHole, symbol Mechanical:MountingHole
- C6, C8, C9: value 10uF -> 1uF
- C7: value 0.1uF -> 1uF
- H1, H2: footprint MountingHole:MountingHole_4.3mm_M4 -> (none)
- H3, H4, H5, H6: footprint MountingHole:MountingHole_2.7mm_M2.5 -> (none)
- R16: value 100 -> 10k
- R7: value 1.1k -> 440
Changed lines of the file:
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@@
 			)
 		)
-		(property "Footprint" "MountingHole:MountingHole_4.3mm_M4"
+		(property "Footprint" ""
 			(at 149.86 95.25 0)
 			(hide yes)
@@
 			)
 		)
-		(property "Value" "10uF"
+		(property "Value" "1uF"
 			(at 121.412 55.118 0)
 			(show_name no)
@@
 			)
 		)
-		(property "Footprint" "MountingHole:MountingHole_2.7mm_M2.5"
+		(property "Footprint" ""
 			(at 149.86 119.38 0)
 			(hide yes)
@@
 			)
 		)
-		(property "Value" "10uF"
+		(property "Value" "1uF"
 			(at 167.64 54.102 0)
 			(show_name no)
@@
 			)
 		)
-		(property "Footprint" "MountingHole:MountingHole_4.3mm_M4"
+		(property "Footprint" ""
 			(at 149.86 101.6 0)
 			(hide yes)
@@
 			)
 		)
-		(property "Footprint" "MountingHole:MountingHole_2.7mm_M2.5"
+		(property "Footprint" ""
 			(at 149.86 125.73 0)
 			(hide yes)
@@
 			)
 		)
-		(property "Value" "0.1uF"
+		(property "Value" "1uF"
 			(at 130.81 62.992 0)
 			(show_name no)
@@
 	)
 	(symbol
+		(lib_id "Mechanical:MountingHole")
+		(at 149.86 139.7 0)
+		(unit 1)
+		(body_style 1)
+		(exclude_from_sim no)
+		(in_bom no)
+		(on_board yes)
+		(in_pos_files yes)
+		(dnp no)
+		(fields_autoplaced yes)
+		(property "Reference" "H8"
+			(at 152.4 138.4299 0)
+			(show_name no)
+			(do_not_autoplace no)
+			(effects
+				(font
+					(size 1.27 1.27)
+				)
+				(justify left)
+			)
+		)
+		(property "Value" "MountingHole"
+			(at 152.4 140.9699 0)
+			(show_name no)
+			(do_not_autoplace no)
+			(effects
+				(font
+					(size 1.27 1.27)
+				)
+				(justify left)
+			)
+		)
+		(property "Footprint" ""
+			(at 149.86 139.7 0)
+			(hide yes)
+			(show_name no)
+			(do_not_autoplace no)
+			(effects
+				(font
+					(size 1.27 1.27)
+				)
+			)
+		)
+		(property "Datasheet" ""
+			(at 149.86 139.7 0)
+			(hide yes)
+			(show_name no)
+			(do_not_autoplace no)
+			(effects
+				(font
+					(size 1.27 1.27)
+				)
+			)
+		)
+		(property "Description" "Mounting Hole without connection"
+			(at 149.86 139.7 0)
+			(hide yes)
+			(show_name no)
+			(do_not_autoplace no)
+			(effects
+				(font
+					(size 1.27 1.27)
+				)
+			)
+		)
+		(instances
+			(project "SilentAlarmClockPCB_V1"
+				(path "/9e0581d1-a9e9-4515-9473-537630af280a"
+					(reference "H8")
+					(unit 1)
+				)
+			)
+		)
+	)
+	(symbol
 		(lib_id "power:GND")
 		(at 152.4 33.02 0)
@@
 			)
 		)
-		(property "Footprint" "MountingHole:MountingHole_2.7mm_M2.5"
+		(property "Footprint" ""
 			(at 149.86 106.68 0)
 			(hide yes)
@@
 			)
 		)
-		(property "Footprint" "MountingHole:MountingHole_2.7mm_M2.5"
+		(property "Footprint" ""
 			(at 149.86 113.03 0)
 			(hide yes)
@@
 			)
 		)
-		(property "Value" "1.1k"
+		(property "Value" "440"
 			(at 115.57 116.332 90)
 			(show_name no)
@@
 	)
 	(symbol
+		(lib_id "Mechanical:MountingHole")
+		(at 149.86 132.08 0)
+		(unit 1)
+		(body_style 1)
+		(exclude_from_sim no)
+		(in_bom no)
+		(on_board yes)
+		(in_pos_files yes)
+		(dnp no)
+		(fields_autoplaced yes)
+		(property "Reference" "H7"
+			(at 152.4 130.8099 0)
+			(show_name no)
+			(do_not_autoplace no)
+			(effects
+				(font
+					(size 1.27 1.27)
+				)
+				(justify left)
+			)
+		)
+		(property "Value" "MountingHole"
+			(at 152.4 133.3499 0)
+			(show_name no)
+			(do_not_autoplace no)
+			(effects
+				(font
+					(size 1.27 1.27)
+				)
+				(justify left)
+			)
+		)
+		(property "Footprint" ""
+			(at 149.86 132.08 0)
+			(hide yes)
+			(show_name no)
+			(do_not_autoplace no)
+			(effects
+				(font
+					(size 1.27 1.27)
+				)
+			)
+		)
+		(property "Datasheet" ""
+			(at 149.86 132.08 0)
+			(hide yes)
+			(show_name no)
+			(do_not_autoplace no)
+			(effects
+				(font
+					(size 1.27 1.27)
+				)
+			)
+		)
+		(property "Description" "Mounting Hole without connection"
+			(at 149.86 132.08 0)
+			(hide yes)
+			(show_name no)
+			(do_not_autoplace no)
+			(effects
+				(font
+					(size 1.27 1.27)
+				)
+			)
+		)
+		(instances
+			(project "SilentAlarmClockPCB_V1"
+				(path "/9e0581d1-a9e9-4515-9473-537630af280a"
+					(reference "H7")
+					(unit 1)
+				)
+			)
+		)
+	)
+	(symbol
 		(lib_id "Regulator_Switching:TPS63001")
 		(at 157.48 59.69 0)
@@
 			)
 		)
-		(property "Value" "100"
+		(property "Value" "10k"
 			(at 139.7 54.6099 0)
 			(show_name no)
@@
 			)
 		)
-		(property "Value" "10uF"
+		(property "Value" "1uF"
 			(at 175.006 57.912 0)
 			(show_name no)
